File: Revision History.kicad_sch (KiCad schematic)
At the start: 0 parts

Commit message: Finished preliminary project schematics and architecture
Changed lines of the file:
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@@
 		)
 	)
-	(text_box "[${#}] ${TITLE}"
+	(text_box "[${#}] ${SHEETNAME}"
 		(exclude_from_sim no)
-		(at 80.01 16.51 0)
-		(size 137.16 12.7)
+		(at 80.8228 10.9799 0)
+		(size 137.16 18.3317)
 		(margins 4.4999 4.4999 4.4999 4.4999)
 		(stroke
 			(width -0.0001)
-			(type default)
+			(type solid)
 		)
 		(fill
