File: OBC.kicad_sch (KiCad schematic)
At the start: 5 parts, among them U1 E73-2G4M08S1C, Y1 32.768

Commit message: Minor tweaks
Changed lines of the file:
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@@
 	)
 	(bus_entry
-		(at 195.58 88.9)
-		(size 2.54 2.54)
-		(stroke
-			(width 0)
-			(type default)
-		)
-	)
-	(bus_entry
-		(at 195.58 91.44)
+		(at 198.12 88.9)
+		(size 2.54 2.54)
+		(stroke
+			(width 0)
+			(type default)
+		)
+	)
+	(bus_entry
+		(at 198.12 91.44)
 		(size 2.54 2.54)
 		(stroke
@@
 	)
 	(bus_entry
-		(at 195.58 83.82)
+		(at 198.12 83.82)
 		(size 2.54 2.54)
 		(stroke
@@
 	)
 	(bus_entry
-		(at 195.58 78.74)
+		(at 198.12 78.74)
 		(size 2.54 2.54)
 		(stroke
@@
 	)
 	(bus_entry
-		(at 195.58 93.98)
+		(at 198.12 93.98)
 		(size 2.54 2.54)
 		(stroke
@@
 	)
 	(bus_entry
-		(at 195.58 81.28)
+		(at 198.12 81.28)
 		(size 2.54 2.54)
 		(stroke
@@
 	)
 	(bus_entry
-		(at 195.58 86.36)
+		(at 198.12 86.36)
 		(size 2.54 2.54)
 		(stroke
@@
 	(bus
 		(pts
-			(xy 195.58 93.98) (xy 195.58 76.2)
-		)
-		(stroke
-			(width 0)
-			(type default)
-		)
-	)
-	(wire
-		(pts
-			(xy 198.12 91.44) (xy 201.93 91.44)
+			(xy 198.12 93.98) (xy 198.12 76.2)
+		)
+		(stroke
+			(width 0)
+			(type default)
+		)
+	)
+	(wire
+		(pts
+			(xy 200.66 91.44) (xy 204.47 91.44)
 		)
 		(stroke
@@
 	(wire
 		(pts
-			(xy 198.12 93.98) (xy 201.93 93.98)
+			(xy 200.66 93.98) (xy 204.47 93.98)
 		)
 		(stroke
@@
 	(wire
 		(pts
-			(xy 198.12 96.52) (xy 201.93 96.52)
-		)
-		(stroke
-			(width 0)
-			(type default)
-		)
-	)
-	(wire
-		(pts
-			(xy 198.12 81.28) (xy 201.93 81.28)
+			(xy 200.66 96.52) (xy 204.47 96.52)
+		)
+		(stroke
+			(width 0)
+			(type default)
+		)
+	)
+	(wire
+		(pts
+			(xy 200.66 81.28) (xy 204.47 81.28)
 		)
 		(stroke
@@
 	(wire
 		(pts
-			(xy 198.12 86.36) (xy 201.93 86.36)
+			(xy 200.66 86.36) (xy 204.47 86.36)
 		)
 		(stroke
@@
 	(wire
 		(pts
-			(xy 198.12 83.82) (xy 201.93 83.82)
+			(xy 200.66 83.82) (xy 204.47 83.82)
 		)
 		(stroke
@@
 	(wire
 		(pts
-			(xy 198.12 88.9) (xy 201.93 88.9)
+			(xy 200.66 88.9) (xy 204.47 88.9)
 		)
 		(stroke
@@
 	(global_label "LoRa_MISO"
 		(shape input)
-		(at 201.93 91.44 0)
-		(fields_autoplaced yes)
-		(effects
-			(font
-				(size 1.27 1.27)
-			)
-			(justify left)
-		)
-		(property "Intersheetrefs" "${INTERSHEET_REFS}"
-			(at 215.0751 91.44 0)
+		(at 204.47 91.44 0)
+		(fields_autoplaced yes)
+		(effects
+			(font
+				(size 1.27 1.27)
+			)
+			(justify left)
+		)
+		(property "Intersheetrefs" "${INTERSHEET_REFS}"
+			(at 217.6151 91.44 0)
 			(hide yes)
 			(show_name no)
@@
 	(global_label "LoRa_NSS"
 		(shape input)
-		(at 201.93 81.28 0)
-		(fields_autoplaced yes)
-		(effects
-			(font
-				(size 1.27 1.27)
-			)
-			(justify left)
-		)
-		(property "Intersheetrefs" "${INTERSHEET_REFS}"
-			(at 214.2284 81.28 0)
+		(at 204.47 81.28 0)
+		(fields_autoplaced yes)
+		(effects
+			(font
+				(size 1.27 1.27)
+			)
+			(justify left)
+		)
+		(property "Intersheetrefs" "${INTERSHEET_REFS}"
+			(at 216.7684 81.28 0)
 			(hide yes)
 			(show_name no)
@@
 	(global_label "LoRa_BUSY"
 		(shape input)
-		(at 201.93 96.52 0)
-		(fields_autoplaced yes)
-		(effects
-			(font
-				(size 1.27 1.27)
-			)
-			(justify left)
-		)
-		(property "Intersheetrefs" "${INTERSHEET_REFS}"
-			(at 215.3775 96.52 0)
+		(at 204.47 96.52 0)
+		(fields_autoplaced yes)
+		(effects
+			(font
+				(size 1.27 1.27)
+			)
+			(justify left)
+		)
+		(property "Intersheetrefs" "${INTERSHEET_REFS}"
+			(at 217.9175 96.52 0)
 			(hide yes)
 			(show_name no)
@@
 	(global_label "LoRa_SCK"
 		(shape input)
-		(at 201.93 86.36 0)
-		(fields_autoplaced yes)
-		(effects
-			(font
-				(size 1.27 1.27)
-			)
-			(justify left)
-		)
-		(property "Intersheetrefs" "${INTERSHEET_REFS}"
-			(at 214.2284 86.36 0)
+		(at 204.47 86.36 0)
+		(fields_autoplaced yes)
+		(effects
+			(font
+				(size 1.27 1.27)
+			)
+			(justify left)
+		)
+		(property "Intersheetrefs" "${INTERSHEET_REFS}"
+			(at 216.7684 86.36 0)
 			(hide yes)
 			(show_name no)
@@
 	(global_label "LoRa_RST"
 		(shape input)
-		(at 201.93 83.82 0)
-		(fields_autoplaced yes)
-		(effects
-			(font
-				(size 1.27 1.27)
-			)
-			(justify left)
-		)
-		(property "Intersheetrefs" "${INTERSHEET_REFS}"
-			(at 213.926 83.82 0)
+		(at 204.47 83.82 0)
+		(fields_autoplaced yes)
+		(effects
+			(font
+				(size 1.27 1.27)
+			)
+			(justify left)
+		)
+		(property "Intersheetrefs" "${INTERSHEET_REFS}"
+			(at 216.466 83.82 0)
 			(hide yes)
 			(show_name no)
@@
 	(global_label "LoRa_SW"
 		(shape input)
-		(at 201.93 93.98 0)
-		(fields_autoplaced yes)
-		(effects
-			(font
-				(size 1.27 1.27)
-			)
-			(justify left)
-		)
-		(property "Intersheetrefs" "${INTERSHEET_REFS}"
-			(at 213.1398 93.98 0)
+		(at 204.47 93.98 0)
+		(fields_autoplaced yes)
+		(effects
+			(font
+				(size 1.27 1.27)
+			)
+			(justify left)
+		)
+		(property "Intersheetrefs" "${INTERSHEET_REFS}"
+			(at 215.6798 93.98 0)
 			(hide yes)
 			(show_name no)
@@
 	(global_label "LoRa_MOSI"
 		(shape input)
-		(at 201.93 88.9 0)
-		(fields_autoplaced yes)
-		(effects
-			(font
-				(size 1.27 1.27)
-			)
-			(justify left)
-		)
-		(property "Intersheetrefs" "${INTERSHEET_REFS}"
-			(at 215.0751 88.9 0)
+		(at 204.47 88.9 0)
+		(fields_autoplaced yes)
+		(effects
+			(font
+				(size 1.27 1.27)
+			)
+			(justify left)
+		)
+		(property "Intersheetrefs" "${INTERSHEET_REFS}"
+			(at 217.6151 88.9 0)
 			(hide yes)
 			(show_name no)
@@
 	(hierarchical_label "{LoRa_BUS}"
 		(shape input)
-		(at 195.58 76.2 90)
-		(effects
-			(font
+		(at 198.12 76.2 90)
+		(effects
+			(font

Commit message: Finalized schematic
Parts:
- added J1: I2C, symbol Connector:Conn_01x04_Pin
- added J2: Conn_02x07_Counter_Clockwise, symbol Connector_Generic:Conn_02x07_Counter_Clockwise
- added J6: SWD, Connector_PinHeader_2.54mm:PinHeader_2x03_P2.54mm_Vertical, symbol Connector_Generic:Conn_02x03_Odd_Even
- added J7: RMF, Connector_PinHeader_2.54mm:PinHeader_1x02_P2.54mm_Vertical, symbol Connector:Conn_01x02_Pin
- added SW3: SW_Push, Button_Switch_SMD:SW_Push_1P1T_NO_CK_KMR2, symbol Switch:SW_Push
- added SW5: RST, Button_Switch_SMD:SW_Push_1P1T_NO_CK_KMR2, symbol Switch:SW_Push
Connections:
- net GND: now also J1.4 (Pin_4), J2.13 (Pin_13), J6.5 (Pin_5), J7.2 (Pin_2), SW3.2, SW5.2
- net RMF: now also J7.1 (Pin_1)
- net RST: now also J6.3 (Pin_3), SW5.1
- net SCL: now also J1.1 (Pin_1)
- net SDA: now also J1.2 (Pin_2)
- net SW0: now also SW3.1
- net SWDCLK: now also J6.4 (Pin_4)
- net SWDIO: now also J6.2 (Pin_2)
- new net +3.3V: J1.3 (Pin_3), J2.14 (Pin_14)
- new net +3V3: J6.1 (Pin_1)
- no-connect marks 12 -> 13
