File: CanSat_Devboard.kicad_pcb (KiCad board)
At the start: 4 copper layers, 51 parts, among them IC1 114993390, J1 I2C, J3 Conn_01x03_Pin, J4 USB_C_Receptacle_USB2.0_16P, J5 693071010811, J6 SWD, J7 RMF, J8 GPIO, SW3 SW_Push, SW4 SHPHLD, SW5 RST, U1 E73-2G4M08S1C, U3 SRV05-4, U4 NPM1300-QEAA-R7, Y1 32.768

Commit message: Continued layout and routing
Parts:
- removed NT1, NT2: NetTie_2, Project_Components:Net_tie_1mm
- moved C16 148.0 mm to (154.8, 70.5), turned to 90 degrees
- moved C15 143.4 mm to (143.4, 62.2)
- moved R12 141.8 mm to (143.4, 60.6)
- moved R11 141.1 mm to (143.4, 59.0), turned to 180 degrees
- moved C14 139.5 mm to (148.8, 71.4)
- moved C13 136.1 mm to (138.2, 62.3), turned to -90 degrees
- moved R17 135.6 mm to (138.7, 58.5), turned to 90 degrees
- moved R16 134.7 mm to (140.2, 58.5), turned to 90 degrees
- moved R13 130.3 mm to (139.5, 75.5), turned to -90 degrees
- moved C12 129.1 mm to (135.9, 67.6)
- moved C19 128.0 mm to (133.6, 65.3), turned to -90 degrees
- moved C18 127.3 mm to (135.1, 65.3), turned to -90 degrees
- moved C17 126.6 mm to (136.7, 65.3), turned to -90 degrees
- moved C11 126.3 mm to (135.9, 69.3)
- moved D6 123.8 mm to (142.7, 72.4), turned to -90 degrees
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Connections:
- C14 pad 2: /Project Architecture/Power/PVSS2 -> GND
- C16 pad 1: /Project Architecture/Power/PVSS1 -> GND
- C17 pad 1: /Project Architecture/Power/PVSS1 -> GND
- C18 pad 1: /Project Architecture/Power/PVSS2 -> GND
- R11 pad 1: VSYS -> VMCU
- R12 pad 2: VSYS -> VMCU
- U1 pad 10: RMF -> SCL
- U1 pad 17: unconnected-(U1C-P1.09-Pad17) -> BM_RST
- U1 pad 18: BM_RST -> unconnected-(U1B-P0.04/AIN2-Pad18)
- U1 pad 2: LoRa_RST -> LoRa_SW
- U1 pad 20: SCL -> unconnected-(U1B-P0.12-Pad20)
- U1 pad 22: SDA -> unconnected-(U1B-P0.07-Pad22)
- U1 pad 3: LoRa_NSS -> LoRa_MISO
- U1 pad 32: unconnected-(U1B-P0.20-Pad32) -> RMF
- U1 pad 34: unconnected-(U1B-P0.22-Pad34) -> SW0
- U1 pad 4: LoRa_SCK -> LoRa_MOSI
- U1 pad 6: LoRa_SW -> LoRa_SCK
- U1 pad 7: LoRa_MOSI -> LoRa_RST
- U1 pad 8: LoRa_MISO -> LoRa_NSS
- U1 pad 9: SW0 -> SDA
- U4 pad 2: /Project Architecture/Power/PVSS1 -> GND
- U4 pad 6: /Project Architecture/Power/PVSS2 -> GND
Routing:
- net VBUS: track 5.91 -> 71.5 mm, vias 0 -> 2
- net VBUSOUT: track 0.00 -> 52.5 mm, vias 0 -> 2
- net VSYS: track 0.00 -> 48.5 mm, vias 0 -> 5
- net CC2: track 0.00 -> 48.2 mm, vias 0 -> 4
- net CC1: track 0.00 -> 45.8 mm, vias 0 -> 4
- net VMCU: track 2.89 -> 36.3 mm
- net SCK: track 3.49 -> 27.8 mm
- net MISO: track 4.64 -> 28.6 mm
- net SDA: track 0.00 -> 22.0 mm, vias 0 -> 2
- net MOSI: track 4.58 -> 26.6 mm
- net CS: track 4.19 -> 26.0 mm
- net SCL: track 0.00 -> 20.6 mm, vias 0 -> 2
- net LoRa_SW: track 0.00 -> 18.0 mm
- net BM_RST: track 0.00 -> 16.5 mm, vias 0 -> 2
- net LoRa_MISO: track 0.00 -> 16.2 mm
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
Commit message: Finished PCB design
Parts:
- moved SW3 74.5 mm to (118.8, 111.0), turned to -90 degrees
- moved TP8 53.9 mm to (147.2, 118.2)
- moved J7 53.8 mm to (122.6, 98.7)
- moved J3 51.7 mm to (126.5, 115.4)
- moved TP7 50.8 mm to (152.0, 104.7)
- moved J1 46.4 mm to (118.8, 98.7)
- moved SW5 42.5 mm to (179.1, 80.2), turned to 90 degrees
- moved C11 42.5 mm to (133.1, 111.6)
- moved C12 42.5 mm to (133.1, 110.0)
- moved C13 42.5 mm to (135.4, 104.7)
- moved C16 42.5 mm to (152.0, 112.8)
- moved C18 42.5 mm to (132.3, 107.7)
- moved C3 42.5 mm to (167.0, 97.9)
- moved C4 42.5 mm to (167.0, 99.4)
- moved D4 42.5 mm to (136.7, 114.8)
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Connections:
- J1 pad 1: SCL -> +3.3V
- J1 pad 2: SDA -> GND
- J1 pad 3: +3.3V -> SDA
- J1 pad 4: GND -> SCL
- J4 pad SH: (no net) -> GND
- J8 pad 1: unconnected-(J8-Pin_1-Pad1) -> +3.3V
- J8 pad 10: unconnected-(J8-Pin_10-Pad10) -> 0.15
- J8 pad 11: unconnected-(J8-Pin_11-Pad11) -> 0.07
- J8 pad 12: unconnected-(J8-Pin_12-Pad12) -> 0.12
- J8 pad 13: unconnected-(J8-Pin_13-Pad13) -> 0.04
- J8 pad 14: unconnected-(J8-Pin_14-Pad14) -> 0.08
- J8 pad 2: +3.3V -> GND
- J8 pad 3: unconnected-(J8-Pin_3-Pad3) -> 1.06
- J8 pad 4: GND -> 1.04
- J8 pad 5: unconnected-(J8-Pin_5-Pad5) -> 1.02
- J8 pad 6: unconnected-(J8-Pin_6-Pad6) -> 1.00
- J8 pad 7: unconnected-(J8-Pin_7-Pad7) -> 0.22
- J8 pad 8: unconnected-(J8-Pin_8-Pad8) -> 0.20
- J8 pad 9: unconnected-(J8-Pin_9-Pad9) -> 0.17
- U1 pad 12: unconnected-(U1B-P0.26-Pad12) -> SW0
- U1 pad 14: unconnected-(U1B-P0.06-Pad14) -> RMF
- U1 pad 16: unconnected-(U1B-P0.08-Pad16) -> 0.08
- U1 pad 18: unconnected-(U1B-P0.04/AIN2-Pad18) -> 0.04
- U1 pad 20: unconnected-(U1B-P0.12-Pad20) -> 0.12
- U1 pad 22: unconnected-(U1B-P0.07-Pad22) -> 0.07
- U1 pad 28: unconnected-(U1B-P0.15-Pad28) -> 0.15
- U1 pad 30: unconnected-(U1B-P0.17-Pad30) -> 0.17
- U1 pad 32: RMF -> 0.20
- U1 pad 34: SW0 -> 0.22
- U1 pad 36: unconnected-(U1C-P1.00-Pad36) -> 1.00
- U1 pad 38: unconnected-(U1C-P1.02-Pad38) -> 1.02
- U1 pad 40: unconnected-(U1C-P1.04-Pad40) -> 1.04
- U1 pad 42: unconnected-(U1C-P1.06-Pad42) -> 1.06
Routing:
- net +3.3V: track 11.2 -> 103.0 mm, vias 2 -> 3
- net RST: track 0.00 -> 41.5 mm, vias 0 -> 1
- net SW0: track 0.00 -> 40.6 mm, vias 0 -> 2
- net 0.07: track 0.00 -> 34.7 mm, vias 0 -> 1
- net 0.17: track 0.00 -> 34.6 mm, vias 0 -> 1
- net Net-(U4A-SHPHLD): track 6.82 -> 40.9 mm, vias 1 -> 2
- net 0.22: track 0.00 -> 33.7 mm, vias 0 -> 1
- net 1.02: track 0.00 -> 32.9 mm, vias 0 -> 1
- net 1.06: track 0.00 -> 32.1 mm, vias 0 -> 1
- net 0.15: track 0.00 -> 31.9 mm, vias 0 -> 1
- net 0.04: track 0.00 -> 31.9 mm, vias 0 -> 1
- net 0.20: track 0.00 -> 31.1 mm, vias 0 -> 1
- net 1.00: track 0.00 -> 30.3 mm, vias 0 -> 1
- net 0.12: track 0.00 -> 30.2 mm, vias 0 -> 1
- net 1.04: track 0.00 -> 29.4 mm, vias 0 -> 1
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- added copper zone on B.Cu, net GND
- added copper zone on F.Cu, net GND
- added copper zone on In1.Cu, net GND
- added copper zone on In2.Cu, net GND
Other:
- board outline added: 64.1 x 43.6 mm
- board text removed: "30°"
- board text removed: "3× 120°"
