File: Power.kicad_sch (KiCad schematic)
At the start: 25 parts, among them SW4 SHPHLD, U4 NPM1300-QEAA-R7

Commit message: Minor tweaks
Parts:
- added JP1: Jumper_2_Bridged, symbol Jumper:Jumper_2_Bridged
- L4, L5: footprint Inductor_SMD:L_0805_2012Metric_Pad1.05x1.20mm_HandSolder -> Inductor_SMD:L_1812_4532Metric
- NT1, NT2: footprint NetTie:NetTie-2_SMD_Pad2.0mm -> Project_Components:Net_tie_1mm
Changed lines of the file:
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@@
 			)
 		)
-		(property "Footprint" "Inductor_SMD:L_0805_2012Metric_Pad1.05x1.20mm_HandSolder"
+		(property "Footprint" "Inductor_SMD:L_1812_4532Metric"
 			(at 193.04 63.5 0)
 			(hide yes)
@@
 	)
 	(symbol
+		(lib_id "Jumper:Jumper_2_Bridged")
+		(at 186.69 135.89 0)
+		(unit 1)
+		(body_style 1)
+		(exclude_from_sim no)
+		(in_bom yes)
+		(on_board yes)
+		(in_pos_files yes)
+		(dnp no)
+		(fields_autoplaced yes)
+		(property "Reference" "JP1"
+			(at 186.69 130.81 0)
+			(show_name no)
+			(do_not_autoplace no)
+			(effects
+				(font
+					(size 1.27 1.27)
+				)
+			)
+		)
+		(property "Value" "Jumper_2_Bridged"
+			(at 186.69 133.35 0)
+			(show_name no)
+			(do_not_autoplace no)
+			(effects
+				(font
+					(size 1.27 1.27)
+				)
+			)
+		)
+		(property "Footprint" ""
+			(at 186.69 135.89 0)
+			(hide yes)
+			(show_name no)
+			(do_not_autoplace no)
+			(effects
+				(font
+					(size 1.27 1.27)
+				)
+			)
+		)
+		(property "Datasheet" ""
+			(at 186.69 140.97 0)
+			(hide yes)
+			(show_name no)
+			(do_not_autoplace no)
+			(effects
+				(font
+					(size 1.27 1.27)
+				)
+			)
+		)
+		(property "Description" "Jumper, 2-pole, closed/bridged"
+			(at 186.69 143.51 0)
+			(hide yes)
+			(show_name no)
+			(do_not_autoplace no)
+			(effects
+				(font
+					(size 1.27 1.27)
+				)
+			)
+		)
+		(pin "1"
+		)
+		(pin "2"
+		)
+		(instances
+			(project "CanSat_Devboard"
+				(path "/f9e05184-c88b-4a88-ae9c-ab2bdb32be7c/5d00bd0a-3bbf-46b2-b8c5-f75441fb4350/dd3743eb-d6f5-4249-8948-a675f2376adf"
+					(reference "JP1")
+					(unit 1)
+				)
+			)
+		)
+	)
+	(symbol
 		(lib_id "power:+3.3V")
 		(at 233.68 55.88 270)
@@
 			)
 		)
-		(property "Footprint" "NetTie:NetTie-2_SMD_Pad2.0mm"
+		(property "Footprint" "Project_Components:Net_tie_1mm"
 			(at 160.02 123.19 0)
 			(hide yes)
@@
 			)
 		)
-		(property "Footprint" "Inductor_SMD:L_0805_2012Metric_Pad1.05x1.20mm_HandSolder"
+		(property "Footprint" "Inductor_SMD:L_1812_4532Metric"
 			(at 229.87 60.96 0)
 			(hide yes)
@@
 			)
 		)
-		(property "Footprint" "NetTie:NetTie-2_SMD_Pad2.0mm"
+		(property "Footprint" "Project_Components:Net_tie_1mm"
 			(at 160.02 133.35 0)
 			(hide yes)

Commit message: Finalized schematic
Parts:
- removed JP1: Jumper_2_Bridged, symbol Jumper:Jumper_2_Bridged
- added BT2: 1S Lipo, Connector_JST:JST_XH_B2B-XH-A_1x02_P2.50mm_Vertical, symbol Device:Battery_Cell
- added TP10: VLDO, TestPoint:TestPoint_Pad_D1.0mm, symbol Connector:TestPoint
- added TP7: VMCU, TestPoint:TestPoint_Pad_D1.0mm, symbol Connector:TestPoint
- added TP8: VSYS, TestPoint:TestPoint_Pad_D1.0mm, symbol Connector:TestPoint
- added TP9: 3V3, TestPoint:TestPoint_Pad_D1.0mm, symbol Connector:TestPoint
Connections:
- net +3.3V: now also TP9.1
- net GND: now also BT2.2 (-)
- net VBAT: now also BT2.1 (+)
- net VLDO: now also TP10.1
- net VMCU: now also TP7.1
- net VSYS: now also TP8.1

Commit message: Started PCB layout
Parts:
- removed BT2: 1S Lipo, Connector_JST:JST_XH_B2B-XH-A_1x02_P2.50mm_Vertical, symbol Device:Battery_Cell
- added J3: Conn_01x03_Pin, Connector_JST:JST_XH_B3B-XH-A_1x03_P2.50mm_Vertical, symbol Connector:Conn_01x03_Pin
Connections:
- net GND: now also J3.2 (Pin_2); no longer U4.18 (NTC)
- net VBAT: now also J3.3 (Pin_3)
- new net NTC: J3.1 (Pin_1), U4.18 (NTC)
Changed lines of the file:
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@@
 		)
 	)
+	(global_label "NTC"
+		(shape input)
+		(at 104.14 78.74 180)
+		(fields_autoplaced yes)
+		(effects
+			(font
+				(size 1.27 1.27)
+			)
+			(justify right)
+		)
+		(property "Intersheetrefs" "${INTERSHEET_REFS}"
+			(at 97.5867 78.74 0)
+			(hide yes)
+			(show_name no)
+			(do_not_autoplace no)
+			(effects
+				(font
+					(size 1.27 1.27)
+				)
+				(justify right)
+			)
+		)
+	)
 	(global_label "BM_INT"
 		(shape input)
@@
 		)
 	)
+	(global_label "NTC"
+		(shape input)
+		(at 264.16 133.35 0)
+		(fields_autoplaced yes)
+		(effects
+			(font
+				(size 1.27 1.27)
+			)
+			(justify left)
+		)
+		(property "Intersheetrefs" "${INTERSHEET_REFS}"
+			(at 270.7133 133.35 0)
+			(hide yes)
+			(show_name no)
+			(do_not_autoplace no)
+			(effects
+				(font
+					(size 1.27 1.27)
+				)
+				(justify left)
+			)
+		)
+	)
 	(global_label "SCL"
 		(shape input)
@@
 	(symbol
 		(lib_id "power:GND")
-		(at 256.54 138.43 270)
+		(at 264.16 135.89 90)
 		(unit 1)
 		(body_style 1)
@@
 		(fields_autoplaced yes)
 		(property "Reference" "#PWR026"
-			(at 250.19 138.43 0)
+			(at 270.51 135.89 0)
 			(hide yes)
 			(show_name no)
@@
 		)
 		(property "Value" "GND"
-			(at 251.46 138.43 0)
+			(at 269.24 135.89 0)
 			(hide yes)
 			(show_name no)
@@
 		)
 		(property "Footprint" ""
-			(at 256.54 138.43 0)
+			(at 264.16 135.89 0)
 			(hide yes)
 			(show_name no)
@@
 		)
 		(property "Datasheet" ""
-			(at 256.54 138.43 0)
+			(at 264.16 135.89 0)
 			(hide yes)
 			(show_name no)
@@
 		)
 		(property "Description" "Power symbol creates a global label with name \"GND\" , ground"
-			(at 256.54 138.43 0)
+			(at 264.16 135.89 0)
 			(hide yes)
 			(show_name no)
@@
 	)
 	(symbol
-		(lib_id "Device:Battery_Cell")
-		(at 259.08 138.43 270)
-		(unit 1)
-		(body_style 1)
-		(exclude_from_sim no)
-		(in_bom yes)
-		(on_board yes)
-		(in_pos_files yes)
-		(dnp no)
-		(fields_autoplaced yes)
-		(property "Reference" "BT2"
-			(at 260.9215 130.81 90)
-			(show_name no)
-			(do_not_autoplace no)
-			(effects
-				(font
-					(size 1.27 1.27)
-				)
-			)
-		)
-		(property "Value" "1S Lipo"
-			(at 260.9215 133.35 90)
-			(show_name no)
-			(do_not_autoplace no)
-			(effects
-				(font
-					(size 1.27 1.27)
-				)
-			)
-		)
-		(property "Footprint" "Connector_JST:JST_XH_B2B-XH-A_1x02_P2.50mm_Vertical"
-			(at 260.604 138.43 90)
-			(hide yes)
-			(show_name no)
-			(do_not_autoplace no)
-			(effects
-				(font
-					(size 1.27 1.27)
-				)
-			)
-		)
-		(property "Datasheet" ""
-			(at 260.604 138.43 90)
-			(hide yes)
-			(show_name no)
-			(do_not_autoplace no)
-			(effects
-				(font
-					(size 1.27 1.27)
-				)
-			)
-		)
-		(property "Description" "Single-cell battery"
-			(at 259.08 138.43 0)
-			(hide yes)
-			(show_name no)
-			(do_not_autoplace no)
-			(effects
-				(font
-					(size 1.27 1.27)
-				)
-			)
-		)
-		(property "Sim.Device" "V"
-			(at 259.08 138.43 0)
-			(hide yes)
-			(show_name no)
-			(do_not_autoplace no)
-			(effects
-				(font
-					(size 1.27 1.27)
-				)
-			)
-		)
-		(property "Sim.Type" "DC"
-			(at 259.08 138.43 0)
-			(hide yes)
-			(show_name no)
-			(do_not_autoplace no)
-			(effects
-				(font
-					(size 1.27 1.27)
-				)
-			)
-		)
-		(property "Sim.Pins" "1=+ 2=-"
-			(at 259.08 138.43 0)
-			(hide yes)
-			(show_name no)
-			(do_not_autoplace no)
-			(effects
-				(font
-					(size 1.27 1.27)
-				)
-			)
-		)
-		(pin "1"
-		)
-		(pin "2"
-		)
-		(instances
-			(project "CanSat_Devboard"
-				(path "/f9e05184-c88b-4a88-ae9c-ab2bdb32be7c/5d00bd0a-3bbf-46b2-b8c5-f75441fb4350/dd3743eb-d6f5-4249-8948-a675f2376adf"
-					(reference "BT2")
-					(unit 1)
-				)
-			)
-		)
-	)
-	(symbol
 		(lib_id "Device:NetTie_2")
 		(at 160.02 133.35 0)
@@
 	)
 	(symbol
-		(lib_id "power:GND")
-		(at 104.14 78.74 270)
-		(mirror x)
+		(lib_id "Connector:Conn_01x03_Pin")
+		(at 259.08 135.89 0)
 		(unit 1)
 		(body_style 1)
@@
 		(dnp no)
 		(fields_autoplaced yes)
-		(property "Reference" "#PWR059"
-			(at 97.79 78.74 0)
-			(hide yes)
+		(property "Reference" "J3"
+			(at 259.715 128.27 0)
 			(show_name no)
 			(do_not_autoplace no)
@@
 			)
 		)
-		(property "Value" "GND"
-			(at 99.06 78.74 0)
-			(hide yes)
+		(property "Value" "Conn_01x03_Pin"
+			(at 259.715 130.81 0)
 			(show_name no)
 			(do_not_autoplace no)
@@
 			)
 		)
-		(property "Footprint" ""
-			(at 104.14 78.74 0)
+		(property "Footprint" "Connector_JST:JST_XH_B3B-XH-A_1x03_P2.50mm_Vertical"
+			(at 259.08 135.89 0)
 			(hide yes)
 			(show_name no)
@@
 		)
 		(property "Datasheet" ""
-			(at 104.14 78.74 0)
+			(at 259.08 135.89 0)
 			(hide yes)
 			(show_name no)
@@
 			)
 		)
-		(property "Description" "Power symbol creates a global label with name \"GND\" , ground"
-			(at 104.14 78.74 0)
+		(property "Description" "Generic connector, single row, 01x03, script generated"
+			(at 259.08 135.89 0)
 			(hide yes)
 			(show_name no)
@@
 			)
 		)
+		(pin "2"
+		)
+		(pin "3"
+		)
 		(pin "1"
 		)
@@
 			(project "CanSat_Devboard"
 				(path "/f9e05184-c88b-4a88-ae9c-ab2bdb32be7c/5d00bd0a-3bbf-46b2-b8c5-f75441fb4350/dd3743eb-d6f5-4249-8948-a675f2376adf"
-					(reference "#PWR059")
+					(reference "J3")
 					(unit 1)
 				)

Commit message: Continued layout and routing
Parts:
- removed NT1, NT2: NetTie_2, Project_Components:Net_tie_1mm, symbol Device:NetTie_2
Connections:
- net PVSS1 is gone; now on net GND: C16.1, C17.1, U4.2 (PVSS1)
- net PVSS2 is gone; now on net GND: C14.2, C18.1, U4.6 (PVSS2)
- net VMCU: now also R11.1, R12.2
- net VSYS: no longer R11.1, R12.2

Commit message: Fixed a roouting mistake
Connections:
- net CC1: now also U4.23 (CC1); no longer U4.24 (CC2)
- net CC2: now also U4.24 (CC2); no longer U4.23 (CC1)
Changed lines of the file:
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@@
 	(global_label "CC2"
 		(shape input)
-		(at 185.42 63.5 0)
+		(at 185.42 66.04 0)
 		(fields_autoplaced yes)
 		(effects
@@
 		)
 		(property "Intersheetrefs" "${INTERSHEET_REFS}"
-			(at 192.1547 63.5 0)
+			(at 192.1547 66.04 0)
 			(hide yes)
 			(show_name no)
@@
 	(global_label "CC1"
 		(shape input)
-		(at 185.42 66.04 0)
+		(at 185.42 63.5 0)
 		(fields_autoplaced yes)
 		(effects
@@
 		)
 		(property "Intersheetrefs" "${INTERSHEET_REFS}"
-			(at 192.1547 66.04 0)
+			(at 192.1547 63.5 0)
 			(hide yes)
 			(show_name no)

Commit message: Changed power routing and board color
Parts:
- R16: value 150k -> 500k
Connections:
- net +3.3V: now also C16.2, L5.2, U4.1 (VOUT1); no longer U4.31 (LSOUT2/VOUTLDO2)
- net VMCU: now also C14.1, L4.1, U4.32 (VOUT2); no longer C16.2, L5.2, U4.1 (VOUT1)
- removed net VOUT2: C14.1, L4.1, U4.30 (LSIN2/VINLDO2), U4.32 (VOUT2)
- no-connect marks 3 -> 5
Other:
- note added: "47k -> 1.8V 500k -> 2.7V"
Changed lines of the file:
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@@
 		)
 	)
+	(text "47k -> 1.8V\n500k -> 2.7V"
+		(exclude_from_sim no)
+		(at 206.502 81.534 0)
+		(effects
+			(font
+				(size 1.27 1.27)
+			)
+		)
+	)
 	(text "Load switch mode\n"
 		(exclude_from_sim no)
@@
 		(at 104.14 71.12)
 	)
+	(no_connect
+		(at 104.14 53.34)
+	)
+	(no_connect
+		(at 185.42 50.8)
+	)
 	(bus_entry
 		(at 34.29 41.91)
@@
 		)
 	)
-	(global_label "VOUT2"
-		(shape input)
-		(at 204.47 58.42 0)
-		(fields_autoplaced yes)
-		(effects
-			(font
-				(size 1.27 1.27)
-			)
-			(justify left)
-		)
-		(property "Intersheetrefs" "${INTERSHEET_REFS}"
-			(at 213.3819 58.42 0)
-			(hide yes)
-			(show_name no)
-			(do_not_autoplace no)
-			(effects
-				(font
-					(size 1.27 1.27)
-				)
-				(justify left)
-			)
-		)
-	)
 	(global_label "SW1"
 		(shape input)
@@
 		)
 	)
-	(global_label "VOUT2"
-		(shape input)
-		(at 104.14 53.34 180)
-		(fields_autoplaced yes)
-		(effects
-			(font
-				(size 1.27 1.27)
-			)
-			(justify right)
-		)
-		(property "Intersheetrefs" "${INTERSHEET_REFS}"
-			(at 95.2281 53.34 0)
-			(hide yes)
-			(show_name no)
-			(do_not_autoplace no)
-			(effects
-				(font
-					(size 1.27 1.27)
-				)
-				(justify right)
-			)
-		)
-	)
 	(global_label "BM_INT"
 		(shape input)
@@
 	(symbol
 		(lib_id "power:+3.3V")
-		(at 233.68 55.88 270)
+		(at 204.47 58.42 270)
 		(unit 1)
 		(body_style 1)
@@
 		(fields_autoplaced yes)
 		(property "Reference" "#PWR055"
-			(at 229.87 55.88 0)
+			(at 200.66 58.42 0)
 			(hide yes)
 			(show_name no)
@@
 		)
 		(property "Value" "VMCU"
-			(at 238.76 55.8799 90)
+			(at 209.55 58.4199 90)
 			(show_name no)
 			(do_not_autoplace no)
@@
 		)
 		(property "Footprint" ""
-			(at 233.68 55.88 0)
+			(at 204.47 58.42 0)
 			(hide yes)
 			(show_name no)
@@
 		)
 		(property "Datasheet" ""
-			(at 233.68 55.88 0)
+			(at 204.47 58.42 0)
 			(hide yes)
 			(show_name no)
@@
 		)
 		(property "Description" "Power symbol creates a global label with name \"+3.3V\""
-			(at 233.68 55.88 0)
+			(at 204.47 58.42 0)
 			(hide yes)
 			(show_name no)
@@
 			)
 		)
-		(property "Value" "150k"
+		(property "Value" "500k"
 			(at 195.58 83.82 90)
 			(show_name no)
@@
 	(symbol
 		(lib_id "power:+3.3V")
-		(at 185.42 50.8 270)
+		(at 233.68 55.88 270)
 		(unit 1)
 		(body_style 1)
@@
 		(fields_autoplaced yes)
 		(property "Reference" "#PWR048"
-			(at 181.61 50.8 0)
+			(at 229.87 55.88 0)
 			(hide yes)
 			(show_name no)
@@
 		)
 		(property "Value" "+3.3V"
-			(at 189.23 50.7999 90)
+			(at 237.49 55.8799 90)
 			(show_name no)
 			(do_not_autoplace no)
@@
 		)
 		(property "Footprint" ""
-			(at 185.42 50.8 0)
+			(at 233.68 55.88 0)
 			(hide yes)
 			(show_name no)
@@
 		)
 		(property "Datasheet" ""
-			(at 185.42 50.8 0)
+			(at 233.68 55.88 0)
 			(hide yes)
 			(show_name no)
@@
 		)
 		(property "Description" "Power symbol creates a global label with name \"+3.3V\""
-			(at 185.42 50.8 0)
+			(at 233.68 55.88 0)
 			(hide yes)
 			(show_name no)
